File: multishield.sch (EAGLE design)
At the start: 23 parts, among them J1 7p-2.54-90d, J2 2x16p-2.54, J3 7p-2.54-90d, J4 2x6p-2.54, J5 7p-2.54-90d, J6 7p-2.54-90d, K2 TS-1101F, M1 ARDUINO_R3_ICSP, SW1 SK-12D01, U1 AD595AQ-DIP14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

Commit message: version 2.2 (Led on D13)
Parts:
- renumbered D9 to 13
Connections:
- net D9B: no longer 13.+
- net SCK: now also 13.+
Other:
- note added: "D13"
- note removed: "D9"
Changed lines of the file:
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@@
 <?xml version="1.0" encoding="utf-8"?>
 <!DOCTYPE eagle SYSTEM "eagle.dtd">
-<eagle version="7.5.0">
+<eagle version="7.6.0">
 <drawing>
 <settings>
@@
 <part name="P+8" library="supply1" deviceset="VCC" device=""/>
 <part name="GND14" library="supply1" deviceset="GND" device=""/>
-<part name="D9" library="Seeed-OPL-Diode" deviceset="DIP-LED-RED-RED(2P-D3MM)" device="" value="SR302DC"/>
+<part name="13" library="Seeed-OPL-Diode" deviceset="DIP-LED-RED-RED(2P-D3MM)" device="" value="SR302DC"/>
 <part name="R2" library="Seeed-OPL-Resistor" deviceset="DIP-RES-1K-5%-1/4W(PR-D2.3XL6.5MM)" device="" value="150Ω"/>
 <part name="GND10" library="supply1" deviceset="GND" device=""/>
@@
 <text x="213.36" y="198.12" size="5.08" layer="97" align="bottom-center">Arduino Multishield
 rev. 0</text>
-<text x="95.25" y="135.89" size="1.778" layer="95">D9</text>
+<text x="95.25" y="135.89" size="1.778" layer="95">D13</text>
 </plain>
 <instances>
@@
 <instance part="P+8" gate="VCC" x="290.83" y="8.89" rot="R270"/>
 <instance part="GND14" gate="1" x="290.83" y="19.05" rot="R90"/>
-<instance part="D9" gate="G$1" x="93.98" y="148.59" rot="R90"/>
+<instance part="13" gate="G$1" x="93.98" y="148.59" rot="R90"/>
 <instance part="R2" gate="G$1" x="93.98" y="156.21" rot="R90"/>
 <instance part="GND10" gate="1" x="93.98" y="162.306" rot="R180"/>
@@
 <wire x1="189.23" y1="30.48" x2="288.29" y2="30.48" width="0.1524" layer="91"/>
 <pinref part="J5" gate="G$1" pin="1"/>
-</segment>
-<segment>
-<pinref part="D9" gate="G$1" pin="+"/>
-<wire x1="93.98" y1="144.78" x2="93.98" y2="135.89" width="0.1524" layer="91"/>
 </segment>
 </net>
@@
 <pinref part="J5" gate="G$1" pin="5"/>
 </segment>
+<segment>
+<pinref part="13" gate="G$1" pin="+"/>
+<wire x1="93.98" y1="144.78" x2="93.98" y2="135.89" width="0.1524" layer="91"/>
+</segment>
 </net>
 <net name="SLAVE-RESET" class="0">
@@
 <net name="N$18" class="0">
 <segment>
-<pinref part="D9" gate="G$1" pin="-"/>
+<pinref part="13" gate="G$1" pin="-"/>
 <pinref part="R2" gate="G$1" pin="1"/>
 </segment>

Commit message: Small changes for rev. 2.3
Parts:
- removed C1: 10uF, Seeed-OPL-Capacitor:DIP-CAP-ALUMINUM-47UF-16V(D5-H9MM)
- added C4: 100nf, Seeed-OPL-Capacitor:DIP-CERAMIC-DISC-100NF-50V-Y5V(D5.0MM)
Connections:
- net N$36: now also C4.2; no longer C1.-
- net N$37: now also C4.1; no longer C1.+
Other:
- note added: "Arduino Multishield rev. 2.3"
- note removed: "Arduino Multishield rev. 0"
Changed lines of the file:
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@@
 <?xml version="1.0" encoding="utf-8"?>
 <!DOCTYPE eagle SYSTEM "eagle.dtd">
-<eagle version="7.6.0">
+<eagle version="8.6.1">
 <drawing>
 <settings>
 <setting alwaysvectorfont="no"/>
+<setting keepoldvectorfont="yes"/>
 <setting verticaltext="up"/>
 </settings>
-<grid distance="0.05" unitdist="inch" unit="inch" style="lines" multiple="1" display="no" altdistance="0.01" altunitdist="inch" altunit="inch"/>
+<grid distance="0.1" unitdist="inch" unit="inch" style="lines" multiple="1" display="no" altdistance="0.01" altunitdist="inch" altunit="inch"/>
 <layers>
 <layer number="1" name="Top" color="4" fill="1" visible="no" active="no"/>
@@
 <part name="GND11" library="supply1" deviceset="GND" device=""/>
 <part name="K2" library="Seeed-OPL-Button" deviceset="DIP-BUTTON-FRONT-WHITE(2P-3.4X6MM)" device="" value="TS-1101F"/>
-<part name="C1" library="Seeed-OPL-Capacitor" deviceset="DIP-CAP-ALUMINUM-47UF-16V(D5-H9MM)" device="" value="10uF"/>
 <part name="GND5" library="supply1" deviceset="GND" device=""/>
 <part name="R1" library="Seeed-OPL-Resistor" deviceset="DIP-RES-1K-5%-1/4W(PR-D2.3XL6.5MM)" device="" value="1K"/>
@@
 <part name="GND10" library="supply1" deviceset="GND" device=""/>
 <part name="R4" library="Seeed-OPL-Resistor" deviceset="DIP-RES-4.7K-5%-1/4W(PR-D2.3XL6.5MM)" device="" value="4.7K"/>
+<part name="C4" library="Seeed-OPL-Capacitor" deviceset="DIP-CERAMIC-DISC-100NF-50V-Y5V(D5.0MM)" device="" value="100nf"/>
 </parts>
 <sheets>
@@
 <wire x1="158.75" y1="193.04" x2="158.75" y2="215.9" width="0.1524" layer="97"/>
 <text x="213.36" y="198.12" size="5.08" layer="97" align="bottom-center">Arduino Multishield
-rev. 0</text>
+rev. 2.3</text>
 <text x="95.25" y="135.89" size="1.778" layer="95">D13</text>
 </plain>
@@
 <instance part="GND11" gate="1" x="331.47" y="45.72" rot="R90"/>
 <instance part="K2" gate="G$1" x="317.5" y="45.72" rot="R180"/>
-<instance part="C1" gate="G$1" x="166.37" y="172.72"/>
 <instance part="GND5" gate="1" x="191.77" y="185.42" rot="R180"/>
 <instance part="R1" gate="G$1" x="208.28" y="177.8"/>
@@
 <instance part="GND10" gate="1" x="93.98" y="162.306" rot="R180"/>
 <instance part="R4" gate="G$1" x="207.01" y="151.13" rot="R180"/>
+<instance part="C4" gate="G$1" x="166.37" y="172.72"/>
 </instances>
 <busses>
@@
 <wire x1="96.52" y1="85.09" x2="66.04" y2="85.09" width="0.1524" layer="91"/>
 <wire x1="66.04" y1="85.09" x2="66.04" y2="172.72" width="0.1524" layer="91"/>
-<pinref part="C1" gate="G$1" pin="+"/>
 <wire x1="66.04" y1="172.72" x2="162.56" y2="172.72" width="0.1524" layer="91"/>
+<pinref part="C4" gate="G$1" pin="1"/>
 </segment>
 </net>
@@
 <net name="N$36" class="0">
 <segment>
-<pinref part="C1" gate="G$1" pin="-"/>
 <pinref part="Q2" gate="G$1" pin="C"/>
 <wire x1="170.18" y1="172.72" x2="191.77" y2="172.72" width="0.1524" layer="91"/>
-</segment>
-</net>
+<pinref part="C4" gate="G$1" pin="2"/>
+</segment>
+</net>
